File: breakout_hdmi/breakout_hdmi.kicad_sch (KiCad schematic)
At the start: 0 parts

Commit message: lapod: Add 50p full HDMI breakout board
The first component of the LaPOD, the HDMI breakout board. Takes the 50
pin Rigol connector, and converts it to 4 full HDMI ports.

Signed-off-by: Olliver Schinagl <oliver@schinagl.nl>
Parts:
- added C1, C2, C3, C4: 100 nF, Capacitor_SMD:C_0603_1608Metric_Pad1.08x0.95mm_HandSolder, symbol Device:C
- added H1, H2, H3: MountingHole, MountingHole:MountingHole_2.2mm_M2_DIN965, symbol Mechanical:MountingHole
- added J1, J2, J3, J4: HDMI_A, LCSC:HDMI-SMD_HDMI-19PIN-043, symbol Connector:HDMI_A
- added J5: Conn_02x25, Connector_IDC:IDC-Header_2x25_P2.54mm_Vertical_SMD, symbol Connector_Generic:Conn_02x25_Odd_Even
- added LED1, LED2, LED3, LED4: TC5050RGBF08-3CJH-AF53A, LCSC:LED-SMD_6P-L5.0-W5.0-TL_TC5050RGBF08, symbol LCSC:TC5050RGBF08-3CJH-AF53A
- added R1, R2, R3, R4: 300 Ω, Resistor_SMD:R_0402_1005Metric_Pad0.72x0.64mm_HandSolder, symbol Device:R_Small
- added R5: 100 Ω, Resistor_SMD:R_0805_2012Metric_Pad1.20x1.40mm_HandSolder, symbol Device:R
Connections:
- new net +2V5: J1.16 (SDA), J2.16 (SDA), J3.16 (SDA), J4.16 (SDA), J5.7 (Pin_7)
- new net +4V: J1.18 (+5V), J2.18 (+5V), J3.18 (+5V), J4.18 (+5V), J5.10 (Pin_10), J5.8 (Pin_8)
- new net -2V5: J1.15 (SCL), J2.15 (SCL), J3.15 (SCL), J4.15 (SCL), J5.4 (Pin_4)
- new net CD1+: J1.19 (HPD), LED1.3 (+), LED1.5 (-), LED1.6 (-)
- new net CD1-: J1.14 (UTILITY), LED1.1 (+), LED1.2 (+), LED1.4 (-)
- new net CD2+: J2.19 (HPD), LED2.3 (+), LED2.5 (-), LED2.6 (-)
- new net CD2-: J2.14 (UTILITY), LED2.1 (+), LED2.2 (+), LED2.4 (-)
- new net CD3+: J3.19 (HPD), LED3.3 (+), LED3.5 (-), LED3.6 (-)
- new net CD3-: J3.14 (UTILITY), LED3.1 (+), LED3.2 (+), LED3.4 (-)
- new net CD4+: J4.19 (HPD), LED4.3 (+), LED4.5 (-), LED4.6 (-)
- new net CD4-: J4.14 (UTILITY), LED4.1 (+), LED4.2 (+), LED4.4 (-)
- new net Earth: C1.2, C2.2, C3.2, C4.2, J1.SH, J2.SH, J3.SH, J4.SH, R1.2, R2.2, R3.2, R4.2
- new net GND: C1.1, C2.1, C3.1, C4.1, J1.11 (CKS), J1.17 (GND), J1.2 (D2S), J1.5 (D1S), J1.8 (D0S), J2.11 (CKS), J2.17 (GND), J2.2 (D2S), J2.5 (D1S), J2.8 (D0S), J3.11 (CKS), J3.17 (GND), J3.2 (D2S), J3.5 (D1S), J3.8 (D0S), J4.11 (CKS), J4.17 (GND), J4.2 (D2S), J4.5 (D1S), J4.8 (D0S), J5.11 (Pin_11), J5.2 (Pin_2), J5.20 (Pin_20), J5.21 (Pin_21), J5.3 (Pin_3), J5.30 (Pin_30), J5.31 (Pin_31), J5.40 (Pin_40), J5.41 (Pin_41), J5.50 (Pin_50), J5.9 (Pin_9), R1.1, R2.1, R3.1, R4.1, R5.1
- new net IN0+: J1.10 (CK+), J5.17 (Pin_17)
- new net IN0-: J1.12 (CK-), J5.16 (Pin_16)
- new net IN1+: J1.7 (D0+), J5.18 (Pin_18)
- new net IN1-: J1.9 (D0-), J5.19 (Pin_19)
- new net IN10+: J3.4 (D1+), J5.23 (Pin_23)
- new net IN10-: J3.6 (D1-), J5.22 (Pin_22)
- new net IN11+: J3.1 (D2+), J5.25 (Pin_25)
- new net IN11-: J3.3 (D2-), J5.24 (Pin_24)
- new net IN12+: J4.10 (CK+), J5.33 (Pin_33)
- new net IN12-: J4.12 (CK-), J5.32 (Pin_32)
- new net IN13+: J4.7 (D0+), J5.34 (Pin_34)
- new net IN13-: J4.9 (D0-), J5.35 (Pin_35)
- new net IN14+: J4.4 (D1+), J5.42 (Pin_42)
- new net IN14-: J4.6 (D1-), J5.43 (Pin_43)
- new net IN15+: J4.1 (D2+), J5.44 (Pin_44)
- new net IN15-: J4.3 (D2-), J5.45 (Pin_45)
- new net IN2+: J1.4 (D1+), J5.27 (Pin_27)
- new net IN2-: J1.6 (D1-), J5.26 (Pin_26)
- new net IN3+: J1.1 (D2+), J5.28 (Pin_28)
- new net IN3-: J1.3 (D2-), J5.29 (Pin_29)
- new net IN4+: J2.10 (CK+), J5.37 (Pin_37)
- new net IN4-: J2.12 (CK-), J5.36 (Pin_36)
- new net IN5+: J2.7 (D0+), J5.38 (Pin_38)
- new net IN5-: J2.9 (D0-), J5.39 (Pin_39)
- new net IN6+: J2.4 (D1+), J5.47 (Pin_47)
- new net IN6-: J2.6 (D1-), J5.46 (Pin_46)
- new net IN7+: J2.1 (D2+), J5.48 (Pin_48)
- new net IN7-: J2.3 (D2-), J5.49 (Pin_49)
- new net IN8+: J3.10 (CK+), J5.13 (Pin_13)
- new net IN8-: J3.12 (CK-), J5.12 (Pin_12)
- new net IN9+: J3.7 (D0+), J5.14 (Pin_14)
- new net IN9-: J3.9 (D0-), J5.15 (Pin_15)
- new net VREF0_7: J1.13 (CEC), J2.13 (CEC), J5.6 (Pin_6)
- new net VREF8_15: J3.13 (CEC), J4.13 (CEC), J5.5 (Pin_5)
- new net nP_detect: J5.1 (Pin_1), R5.2
Other:
- note added: "B"
- note added: "G"
- note added: "LOW = board connected"
- note added: "R"
- company: (none) -> Sergey Petrukhin, Peter Lampe, Nikki Smith & Olliver Schinagl
- title: (none) -> LaPOD 50p Full HDMI breakout
