File: pod_sn65lvds/pod_sn65lvds.kicad_sch (KiCad schematic)
At the start: 28 parts, among them J2 Conn_02x04_Odd_Even, U1 SN65LVDS047PW, U2 TLV74325PDBVR

Commit message: fix: Replace SN65LVDS31D/SN65LVDS047W with SN65LVDS391PWR
We accidentally used the incorrect LVDS comparator. The difference is
subtle, but important.

The symbol came from the KiCad default library, the rest of the part
number from LCSC, but was simply the wrong one. 31D vs 391PWR. Subtle
but important.

Luckily, the footprint was almost the same, so no real changes where needed
here.

Signed-off-by: Olliver Schinagl <oliver@schinagl.nl>
Parts:
- removed U1: SN65LVDS047PW, Package_SO:TSSOP-16_4.4x5mm_P0.65mm, symbol Interface:SN65LVDS047PW
- added R12, R13: 1 kΩ, Resistor_SMD:R_0805_2012Metric_Pad1.20x1.40mm_HandSolder, symbol Device:R
- added U1: SN65LVDS391PWR, Package_SO:TSSOP-16_4.4x5mm_P0.65mm, symbol LCSC:SN65LVDS31D
Connections:
- net +3V3: now also R12.1, U1.4 (VCC)
- net GND: now also R13.2, U1.5 (GND)
- net IN0: now also U1.7 (DIN4)
- net IN1: now also U1.6 (DIN3)
- net IN2: now also U1.3 (DIN2)
- net IN3: now also U1.2 (DIN1)
- net OUT0+: now also U1.10 (DOUT4+)
- net OUT0-: now also U1.9 (DOUT4-)
- net OUT1+: now also U1.12 (DOUT3+)
- net OUT1-: now also U1.11 (DOUT3-)
- net OUT2+: now also U1.14 (DOUT2+)
- net OUT2-: now also U1.13 (DOUT2-)
- net OUT3+: now also U1.16 (DOUT1+)
- net OUT3-: now also U1.15 (DOUT1-)
- new net: R12.2, U1.1 (EN1,2)
- new net: R13.1, U1.8 (EN3,4)
Changed lines of the file:
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@@
   (junction (at 45.72 20.32) (diameter 0) (color 0 0 0 0)
-  )
-  (junction (at 57.15 60.96) (diameter 0) (color 0 0 0 0)
   )
   (junction (at 119.38 74.93) (diameter 0) (color 0 0 0 0)
@@
     (stroke (width 0) (type default))
   )
-  (wire (pts (xy 57.15 60.96) (xy 57.15 63.5))
-    (stroke (width 0) (type default))
-  )
   (wire (pts (xy 45.72 20.32) (xy 45.72 22.86))
     (stroke (width 0) (type default))
@@
     (stroke (width 0) (type default))
   )
+  (wire (pts (xy 77.47 68.58) (xy 77.47 71.12))
+    (stroke (width 0) (type default))
+  )
   (wire (pts (xy 171.45 100.33) (xy 171.45 92.71))
     (stroke (width 0) (type default))
@@
     (stroke (width 0) (type default))
   )
+  (wire (pts (xy 52.07 29.21) (xy 52.07 60.96))
+    (stroke (width 0) (type default))
+  )
   (wire (pts (xy 148.59 69.85) (xy 148.59 95.25))
     (stroke (width 0) (type default))
@@
     (stroke (width 0) (type default))
   )
-  (wire (pts (xy 52.07 60.96) (xy 57.15 60.96))
+  (wire (pts (xy 52.07 60.96) (xy 62.23 60.96))
     (stroke (width 0) (type default))
   )
@@
     (stroke (width 0) (type default))
   )
-  (wire (pts (xy 77.47 71.12) (xy 77.47 68.58))
-    (stroke (width 0) (type default))
-  )
   (wire (pts (xy 151.13 21.59) (xy 151.13 59.69))
     (stroke (width 0) (type default))
@@
     (stroke (width 0) (type default))
   )
-  (wire (pts (xy 57.15 63.5) (xy 62.23 63.5))
-    (stroke (width 0) (type default))
-  )
   (wire (pts (xy 19.05 55.88) (xy 29.21 55.88))
     (stroke (width 0) (type default))
@@
     (stroke (width 0) (type default))
   )
+  (wire (pts (xy 59.69 63.5) (xy 62.23 63.5))
+    (stroke (width 0) (type default))
+  )
   (wire (pts (xy 118.11 36.83) (xy 118.11 39.37))
     (stroke (width 0) (type default))
@@
     (stroke (width 0) (type default))
   )
-  (wire (pts (xy 57.15 60.96) (xy 62.23 60.96))
-    (stroke (width 0) (type default))
-  )
   (wire (pts (xy 39.37 38.1) (xy 39.37 43.18))
     (stroke (width 0) (type default))
@@
     (stroke (width 0) (type default))
   )
-  (wire (pts (xy 52.07 20.32) (xy 52.07 60.96))
+  (wire (pts (xy 52.07 20.32) (xy 52.07 21.59))
     (stroke (width 0) (type default))
   )
@@
     )
   )
+  (symbol (lib_id "Device:R") (at 52.07 25.4 0) (unit 1)
+    (in_bom yes) (on_board yes) (dnp no)
+    (property "Reference" "R12" (at 54.61 24.13 0)
+      (effects (font (size 1.27 1.27)) (justify left))
+    )
+    (property "Value" "1 kΩ" (at 54.61 26.67 0)
+      (effects (font (size 1.27 1.27)) (justify left))
+    )
+    (property "Footprint" "Resistor_SMD:R_0805_2012Metric_Pad1.20x1.40mm_HandSolder" (at 50.292 25.4 90)
+      (effects (font (size 1.27 1.27)) hide)
+    )
+    (property "Datasheet" "~" (at 52.07 25.4 0)
+      (effects (font (size 1.27 1.27)) hide)
+    )
+    (property "LCSC" "C17513" (at 52.07 25.4 0)
+      (effects (font (size 1.27 1.27)) hide)
+    )
+    (property "package" "0805" (at 52.07 25.4 0)
+      (effects (font (size 1.27 1.27)) hide)
+    )
+    (property "power" "125 mW" (at 52.07 25.4 0)
+      (effects (font (size 1.27 1.27)) hide)
+    )
+    (property "tolerance" "1%" (at 52.07 25.4 0)
+      (effects (font (size 1.27 1.27)) hide)
+    )
+    (pin "1")
+    (pin "2")
+    (instances
+      (project "pod_sn65lvds"
+        (path "/f60f0a6c-68c3-494b-b6bb-e80732df7e71"
+          (reference "R12") (unit 1)
+        )
+      )
+    )
+  )
   (symbol (lib_id "power:+4V") (at 19.05 35.56 0) (mirror y) (unit 1)
     (in_bom yes) (on_board yes) (dnp no)
@@
         (path "/f60f0a6c-68c3-494b-b6bb-e80732df7e71"
           (reference "#PWR017") (unit 1)
-        )
-      )
-    )
-  )
-  (symbol (lib_id "Interface:SN65LVDS047PW") (at 77.47 45.72 0) (unit 1)
-    (in_bom yes) (on_board yes) (dnp no) (fields_autoplaced)
-    (property "Reference" "U1" (at 79.6641 20.32 0)
-      (effects (font (size 1.27 1.27)) (justify left))
-    )
-    (property "Value" "SN65LVDS047PW" (at 79.6641 22.86 0)
-      (effects (font (size 1.27 1.27)) (justify left))
-    )
-    (property "Footprint" "Package_SO:TSSOP-16_4.4x5mm_P0.65mm" (at 74.93 69.85 0)
-      (effects (font (size 1.27 1.27)) hide)
-    )
-    (property "Datasheet" "docs/1912111437_Texas-Instruments-SN65LVDS31D_C352934.pdf" (at 78.74 45.72 0)
-      (effects (font (size 1.27 1.27)) hide)
-    )
-    (property "LCSC" "C114984" (at 77.47 45.72 0)
-      (effects (font (size 1.27 1.27)) hide)
-    )
-    (pin "1")
-    (pin "10")
-    (pin "11")
-    (pin "12")
-    (pin "13")
-    (pin "14")
-    (pin "15")
-    (pin "16")
-    (pin "2")
-    (pin "3")
-    (pin "4")
-    (pin "5")
-    (pin "6")
-    (pin "7")
-    (pin "8")
-    (pin "9")
-    (instances
-      (project "pod_sn65lvds"
-        (path "/f60f0a6c-68c3-494b-b6bb-e80732df7e71"
-          (reference "U1") (unit 1)
         )
       )
@@
     )
   )
+  (symbol (lib_id "power:GND") (at 59.69 71.12 0) (unit 1)
+    (in_bom yes) (on_board yes) (dnp no) (fields_autoplaced)
+    (property "Reference" "#PWR024" (at 59.69 77.47 0)
+      (effects (font (size 1.27 1.27)) hide)
+    )
+    (property "Value" "GND" (at 59.69 76.2 0)
+      (effects (font (size 1.27 1.27)))
+    )
+    (property "Footprint" "" (at 59.69 71.12 0)
+      (effects (font (size 1.27 1.27)) hide)
+    )
+    (property "Datasheet" "" (at 59.69 71.12 0)
+      (effects (font (size 1.27 1.27)) hide)
+    )
+    (pin "1")
+    (instances
+      (project "pod_sn65lvds"
+        (path "/f60f0a6c-68c3-494b-b6bb-e80732df7e71"
+          (reference "#PWR024") (unit 1)
+        )
+      )
+    )
+  )
+  (symbol (lib_id "Device:R") (at 59.69 67.31 0) (mirror y) (unit 1)
+    (in_bom yes) (on_board yes) (dnp no) (fields_autoplaced)
+    (property "Reference" "R13" (at 57.15 66.04 0)
+      (effects (font (size 1.27 1.27)) (justify left))
+    )
+    (property "Value" "1 kΩ" (at 57.15 68.58 0)
+      (effects (font (size 1.27 1.27)) (justify left))
+    )
+    (property "Footprint" "Resistor_SMD:R_0805_2012Metric_Pad1.20x1.40mm_HandSolder" (at 61.468 67.31 90)
+      (effects (font (size 1.27 1.27)) hide)
+    )
+    (property "Datasheet" "~" (at 59.69 67.31 0)
+      (effects (font (size 1.27 1.27)) hide)
+    )
+    (property "LCSC" "C17513" (at 59.69 67.31 0)
+      (effects (font (size 1.27 1.27)) hide)
+    )
+    (property "package" "0805" (at 59.69 67.31 0)
+      (effects (font (size 1.27 1.27)) hide)
+    )
+    (property "power" "125 mW" (at 59.69 67.31 0)
+      (effects (font (size 1.27 1.27)) hide)
+    )
+    (property "tolerance" "1%" (at 59.69 67.31 0)
+      (effects (font (size 1.27 1.27)) hide)
+    )
+    (pin "1")
+    (pin "2")
+    (instances
+      (project "pod_sn65lvds"
+        (path "/f60f0a6c-68c3-494b-b6bb-e80732df7e71"
+          (reference "R13") (unit 1)
+        )
+      )
+    )
+  )
   (symbol (lib_id "Device:LED") (at 119.38 80.01 270) (mirror x) (unit 1)
     (in_bom yes) (on_board yes) (dnp no)
@@
         )
       )
+    )
+  )
+  (symbol (lib_id "LCSC:SN65LVDS31D") (at 77.47 43.18 0) (unit 1)
+    (in_bom yes) (on_board yes) (dnp no)
+    (property "Reference" "U1" (at 66.04 24.13 0)
+      (effects (font (size 1.27 1.27)))
+    )
+    (property "Value" "SN65LVDS391PWR" (at 86.36 24.13 0)
+      (effects (font (size 1.27 1.27)))
+    )
+    (property "Footprint" "Package_SO:TSSOP-16_4.4x5mm_P0.65mm" (at 77.47 59.69 0)
+      (effects (font (size 1.27 1.27)) hide)
+    )
+    (property "Datasheet" "docs/2303021200_Texas-Instruments-SN65LVDS391PWR_C354139.pdf" (at 77.47 62.23 0)
+      (effects (font (size 1.27 1.27)) hide)
+    )
+    (property "LCSC" "C354139" (at 77.47 43.18 0)
+      (effects (font (size 1.27 1.27)) hide)
+    )
+    (property "tolerance" "" (at 77.47 43.18 0)
+      (effects (font (size 1.27 1.27)) hide)
+    )
+    (property "voltage" "" (at 77.47 43.18 0)
+      (effects (font (size 1.27 1.27)) hide)
+    )
+    (property "power" "" (at 77.47 43.18 0)
+      (effects (font (size 1.27 1.27)) hide)
+    )
+    (property "temp_coef" "" (at 77.47 43.18 0)
+      (effects (font (size 1.27 1.27)) hide)
+    )
+    (property "package" "" (at 77.47 43.18 0)
+      (effects (font (size 1.27 1.27)) hide)
+    )
+    (pin "7")
+    (pin "11")
+    (pin "8")
+    (pin "3")
+    (pin "2")
+    (pin "9")
+    (pin "5")
+    (pin "4")
+    (pin "13")
+    (pin "14")
+    (pin "15")
+    (pin "1")
+    (pin "12")
+    (pin "6")
+    (pin "16")
+    (pin "10")
+    (instances
+      (project "pod_sn65lvds"
+        (path "/f60f0a6c-68c3-494b-b6bb-e80732df7e71"
+          (reference "U1") (unit 1)
+        )
+      )
